File: Boost/eagle/Boost.brd (EAGLE design)
At the start: 66 x 61 mm, 21 parts, among them X1 22-23-2051, X2 22-23-2021

Commit message: boost: change resistor values
Parts:
- R1, R2: value (none) -> 0
- R3, R4: value (none) -> 10k
Changed lines of the file:
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@@
 <attribute name="MPN" value="7447709150" x="18.415" y="45.085" size="1.778" layer="27" display="off"/>
 </element>
-<element name="R1" library="resistor" package="MINI_MELF-0204W" value="" x="38.735" y="33.655" rot="MR0"/>
-<element name="R2" library="resistor" package="MINI_MELF-0204W" value="" x="41.275" y="26.67" rot="MR0"/>
-<element name="R3" library="resistor" package="MINI_MELF-0204W" value="" x="33.02" y="30.48" rot="MR180"/>
-<element name="R4" library="resistor" package="MINI_MELF-0204W" value="" x="36.195" y="26.67" rot="MR90"/>
+<element name="R1" library="resistor" package="MINI_MELF-0204W" value="0" x="38.735" y="33.655" rot="MR0"/>
+<element name="R2" library="resistor" package="MINI_MELF-0204W" value="0" x="41.275" y="26.67" rot="MR0"/>
+<element name="R3" library="resistor" package="MINI_MELF-0204W" value="10k" x="33.02" y="30.48" rot="MR180"/>
+<element name="R4" library="resistor" package="MINI_MELF-0204W" value="10k" x="36.195" y="26.67" rot="MR90"/>
 <element name="U$1" library="ppst002" package="D-PAK" value="IRLR7807" x="33.02" y="29.21" rot="R180"/>
 <element name="U$2" library="ppst002" package="D-PAK" value="IRLR7807" x="25.4" y="31.75"/>
